Commit message: [ros | os1_64_bauzil] Add rviz node use xacro for robot spawn

File: urdf/os1_64.urdf.xacro (robot description, xacro)
@@ -2,6 +2,7 @@
 <robot xmlns:xacro="http://www.ros.org/wiki/xacro" name="os1_64">
   <xacro:property name="PI" value="3.1415926535897931"/>
-  <xacro:macro name="OS1-64" params="*origin parent:=base_link name:=ouster topic:=/points hz:=10 samples:=512 min_range:=0.8 max_range:=100 noise:=0.008 min_angle_v:=-16.6 max_angle_v:=16.6">
+  <xacro:macro name="os1_64" params="*origin parent:=base_link name:=ouster topic:=/points hz:=10 samples:=512 min_range:=0.8 max_range:=100 noise:=0.008 min_angle_v:=-16.6 max_angle_v:=16.6">
     <joint name="${name}_base_mount_joint" type="fixed">
+      <xacro:insert_block name="origin" />
       <parent link="${parent}"/>
       <child link="${name}"/>
@@ -21,7 +22,7 @@
       </collision>
       <visual name="base_visual">
-        <origin xyz="0 0 -0.03675" rpy="0 0 0" />
+        <origin xyz="0 0 -0.03675" rpy="0 0 0"/>
         <geometry>
-          <mesh filename="package://os1_64_bauzil/sdf_data/os1_64.stl" />
+          <mesh filename="package://os1_64_bauzil/sdf/data/os1_64.stl"/>
         </geometry>
       </visual>
@@ -37,12 +38,12 @@
               <samples>64</samples>
               <resolution>1</resolution>
-              <min_angle>-${min_angle_v*M_PI/180.0}</min_angle>
-              <max_angle> ${max_angle_v*M_PI/180.0}</max_angle>
+              <min_angle>${min_angle_v*PI/180.0}</min_angle>
+              <max_angle>${max_angle_v*PI/180.0}</max_angle>
             </vertical>
             <horizontal>
               <samples>${samples}</samples>
               <resolution>1</resolution>
-              <min_angle>-${M_PI}</min_angle>
-              <max_angle>${M_PI}</max_angle>
+              <min_angle>-${PI}</min_angle>
+              <max_angle>${PI}</max_angle>
             </horizontal>
           </scan>

Commit message: [ros | os1_64_bauzil] minor changes for ros topics

File: urdf/os1_64.urdf.xacro (robot description, xacro)
@@ -2,5 +2,5 @@
 <robot xmlns:xacro="http://ros.org/wiki/xacro" name="os1_64">
   <xacro:property name="PI" value="3.1415926535897931"/>
-  <xacro:macro name="os1_64" params="*origin parent:=base_link name:=ouster topic:=/points hz:=10 samples:=512 min_range:=0.8 max_range:=100 noise:=0.008 min_angle_v:=-16.6 max_angle_v:=16.6">
+  <xacro:macro name="os1_64" params="*origin parent:=base_link name:=ouster prefix:=/os1_cloud_node hz:=10 samples:=512 min_range:=0.8 max_range:=100 noise:=0.008 min_angle_v:=-16.6 max_angle_v:=16.6">
     <joint name="${name}_base_mount_joint" type="fixed">
       <xacro:insert_block name="origin" />
@@ -29,6 +29,6 @@
     </link>
     <gazebo reference="${name}">
-      <sensor type="ray" name="${name}-lidar">
-        <pose>0 0 0 0 0 0</pose>
+      <sensor type="ray" name="${name}_lidar">
+        <pose>0 0 0 0 0 ${PI}</pose>
         <visualize>false</visualize>
         <update_rate>${hz}</update_rate>
@@ -60,5 +60,5 @@
         </ray>
         <plugin name="gazebo_ros_laser_controller" filename="libgazebo_ros_ouster_laser.so">
-          <topicName>${topic}</topicName>
+          <topicName>${prefix}/points</topicName>
           <frameName>${name}</frameName>
           <min_range>${min_range}</min_range>
@@ -68,4 +68,27 @@
       </sensor>
     </gazebo>
+    <link name="${name}_imu"/>
+    <joint name="${name}_imu_joint" type="fixed">
+      <parent link="${name}"/>
+      <child link="${name}_imu"/>
+    </joint>
+    <gazebo reference="${name}_imu">
+      <sensor type="imu" name="${name}_imu_sensor">
+        <pose>0 0 0 0 0 0</pose>
+        <always_on>true</always_on>
+        <update_rate>100</update_rate>
+        <visualize>true</visualize>
+        <topic>${prefix}/imu</topic>
+        <!-- <plugin filename="libgazebo_ros_imu_sensor.so" name="imu_plugin">
+          <topicName>${prefix}/imu</topicName>
+          <bodyName>os1_imu</bodyName>
+          <updateRateHZ>100.0</updateRateHZ>
+          <gaussianNoise>0.0</gaussianNoise>
+          <xyzOffset>0 0 0</xyzOffset>
+          <rpyOffset>0 0 0</rpyOffset>
+          <frameName>os1_imu</frameName>
+        </plugin> -->
+      </sensor>
+    </gazebo>
   </xacro:macro>
 </robot>

File: urdf/talos_full_v2_sensors.urdf.xacro (robot description, xacro)
@@ -47,5 +47,6 @@
   <xacro:include filename="$(find talos_data)/urdf/materials.urdf.xacro" />
   <xacro:include filename="$(find os1_64_bauzil)/urdf/os1_64.urdf.xacro"/>
-  <os1_64 parent="head_2_link" name="ouster" topic="/os1_cloud_node/points" hz="10" samples="512">
+  <!-- noise:=0.0 means that the noise is calculated according to the datasheet -->
+  <os1_64 parent="head_2_link" name="os1" prefix="/os1_cloud_node" hz="10" samples="512" noise="0.0">
     <origin xyz="0 0 0.312" rpy="0 0 1.570796327"/>
   </os1_64>

Commit message: [ros | os1_64_bauzil] error on os model

File: urdf/os1_64.urdf.xacro (robot description, xacro)
@@ -22,5 +22,5 @@
       </collision>
       <visual name="base_visual">
-        <origin xyz="0 0 -0.03675" rpy="0 0 0"/>
+        <origin xyz="0 0 0" rpy="0 0 0"/>
         <geometry>
           <mesh filename="package://os1_64_bauzil/sdf/data/os1_64.stl"/>

File: urdf/talos_full_v2_sensors.urdf.xacro (robot description, xacro)
@@ -49,5 +49,5 @@
   <!-- noise:=0.0 means that the noise is calculated according to the datasheet -->
   <os1_64 parent="head_2_link" name="os1" prefix="/os1_cloud_node" hz="10" samples="512" noise="0.0">
-    <origin xyz="0 0 0.312" rpy="0 0 1.570796327"/>
+    <origin xyz="0 0 0.275" rpy="0 0 1.570796327"/>
   </os1_64>
 </robot>

Commit message: correct package name

File: urdf/os1_64.urdf.xacro (robot description, xacro)
@@ -24,5 +24,5 @@
         <origin xyz="0 0 0" rpy="0 0 0"/>
         <geometry>
-          <mesh filename="package://os1_64_bauzil/sdf/data/os1_64.stl"/>
+          <mesh filename="package://talos_bauzil/sdf/data/os1_64.stl"/>
         </geometry>
       </visual>

File: urdf/robot.urdf.xacro (robot description, xacro)
@@ -28,5 +28,5 @@
     </inertial>
   </link>
-  <xacro:include filename="$(find os1_64_bauzil)/urdf/os1_64.urdf.xacro"/>
+  <xacro:include filename="$(find talos_bauzil)/urdf/os1_64.urdf.xacro"/>
   <os1_64 parent="base_link" name="ouster" topic="/os1_cloud_node/points" hz="10" samples="512">
     <origin xyz="0 0 1." rpy="0 0 0" />
