Commit message: Add info on xacros

File: urdf/head/head_ouster.urdf.xacro (robot description, xacro)
@@ -6,4 +6,8 @@
   To view a copy of this license, visit http://creativecommons.org/licenses/by-nc-nd/3.0/ or send a letter to
   Creative Commons, 444 Castro Street, Suite 900, Mountain View, California, 94041, USA.
+-->
+<!--
+  Extracted from robotpkg-talos-data/urdf/head.
+  Modified by T. Lasguignes, LAAS-CNRS.
 -->
 <robot xmlns:xacro="http://ros.org/wiki/xacro">
@@ -107,5 +111,8 @@
     </gazebo>
   </xacro:macro>
-  <xacro:macro name="talos_head" params="name parent">
+  <!--************************-->
+  <!--          Head          -->
+  <!--************************-->
+  <xacro:macro name="talos_head" params="name parent lid_samples:=512 lid_hz:=10">
     <xacro:talos_head_1 name="${name}_1" parent="${parent}" />
     <xacro:talos_head_2 name="${name}_2" parent="${name}_1_link"/>
@@ -121,5 +128,5 @@
                                                 offset_value_1="${head_1_joint_offset}" offset_value_2="${head_2_joint_offset}"/>
     <!-- noise:=0.0 means that the noise is calculated according to the datasheet -->
-    <xacro:os1_64 parent="${name}_2" name="os1" prefix="/os1_cloud_node" hz="10" samples="512" noise="0.0" gpu="true" reduced="false">
+    <xacro:os1_64 parent="${name}_2" name="os1" prefix="/os1_cloud_node" hz="${lid_hz}" samples="${lid_samples}" noise="0.0" gpu="true" reduced="false">
       <origin xyz="0 0 0.275" rpy="0 0 0"/>
     </xacro:os1_64>

File: urdf/talos_full_v2_ouster.urdf.xacro (robot description, xacro)
@@ -6,4 +6,8 @@
   To view a copy of this license, visit http://creativecommons.org/licenses/by-nc-nd/3.0/ or send a letter to
   Creative Commons, 444 Castro Street, Suite 900, Mountain View, California, 94041, USA.
+-->
+<!--
+  Extracted from robotpkg-talos-data/robots.
+  Modified by T. Lasguignes, LAAS-CNRS.
 -->
 <robot name="talos" xmlns:xacro="http://ros.org/wiki/xacro"
@@ -15,5 +19,5 @@
   </xacro:if>
   <xacro:include filename="$(find talos_data)/urdf/torso/torso.urdf.xacro" />
-  <xacro:include filename="$(find talos_data)/urdf/head/head.urdf.xacro" />
+  <xacro:include filename="$(find talos_bauzil)/urdf/head/head_ouster.urdf.xacro" /> <!--modif-->
   <!--arm_v1 loadded because of the different joint range for 1st DoF-->
   <xacro:include filename="$(find talos_data)/urdf/arm/arm_v2.urdf.xacro" />
@@ -33,5 +37,5 @@
     <xacro:crane parent="torso_2_link"/>
   </xacro:if>
-  <xacro:talos_head name="head" parent="torso_2_link"/>
+  <xacro:talos_head name="head" parent="torso_2_link" lid_samples="1024"/>
   <xacro:talos_arm name="arm" parent="torso_2_link" side="left" reflect="1"/>
   <xacro:talos_arm name="arm" parent="torso_2_link" side="right" reflect="-1"/>
@@ -46,8 +50,3 @@
   <!-- Materials for visualization -->
   <xacro:include filename="$(find talos_data)/urdf/materials.urdf.xacro" />
-  <xacro:include filename="$(find ouster_os1_64)/urdf/os1_64.urdf.xacro"/>
-  <!-- noise:=0.0 means that the noise is calculated according to the datasheet -->
-  <os1_64 parent="head_2" name="os1" prefix="/os1_cloud_node" hz="10" samples="512" noise="0.0" gpu="true" reduced="false">
-    <origin xyz="0 0 0.275" rpy="0 0 0"/>
-  </os1_64>
 </robot>
